File: lineScope-05A-probe.kicad_pcb (KiCad board)
At the start: 2 copper layers, 99.5 x 30 mm, 25 parts, among them J4 Conn_01x03, T1 TA1310-03

Commit message: Minor Update
Connections:
- net /HV_{L} renamed /HV_{LIN}
- net /HV_{N} renamed /HV_{LOUT}
- net Net-(J4-Pin_1) renamed /OUT_{H}
- net Net-(J4-Pin_3) renamed /OUT_{L}
Changed lines of the file:
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@@
 	(net 7 "Net-(H4-Pad1)")
 	(net 8 "/HV_{L1}")
-	(net 9 "/HV_{L}")
-	(net 10 "/HV_{N}")
-	(net 11 "Net-(J4-Pin_3)")
-	(net 12 "Net-(J4-Pin_1)")
+	(net 9 "/HV_{LIN}")
+	(net 10 "/HV_{LOUT}")
+	(net 11 "/OUT_{L}")
+	(net 12 "/OUT_{H}")
 	(footprint "Koszalix_Transformers:PowerUC-TA1310-03"
 		(layer "F.Cu")
@@
 			)
 		)
-		(property "Datasheet" ""
+		(property "Datasheet" "https://cdn.shopifycdn.net/s/files/1/2723/6858/files/TA1310.pdf?v=1652424066"
 			(at 0 0 90)
 			(unlocked yes)
@@
 			)
 		)
+		(sheetname "Root")
+		(sheetfile "lineScope-05A-probe.kicad_sch")
 		(attr through_hole)
 		(fp_rect
@@
 			(layers "*.Cu" "*.Mask")
 			(remove_unused_layers no)
-			(net 10 "/HV_{N}")
+			(net 10 "/HV_{LOUT}")
 			(pintype "passive")
 		)
@@
 			)
 		)
+		(sheetname "Root")
+		(sheetfile "lineScope-05A-probe.kicad_sch")
 		(attr through_hole)
 		(fp_rect
@@
 			(layers "*.Cu" "*.Mask")
 			(remove_unused_layers no)
-			(net 10 "/HV_{N}")
+			(net 10 "/HV_{LOUT}")
 			(pintype "passive")
 		)
@@
 			(layers "*.Cu" "*.Mask")
 			(remove_unused_layers no)
-			(net 10 "/HV_{N}")
+			(net 10 "/HV_{LOUT}")
 			(pintype "passive")
 		)
@@
 			(layers "F.Cu" "F.Paste" "F.Mask")
 			(roundrect_rratio 0.192308)
-			(net 11 "Net-(J4-Pin_3)")
+			(net 11 "/OUT_{L}")
 			(pintype "passive")
 		)
@@
 			)
 		)
+		(sheetname "Root")
+		(sheetfile "lineScope-05A-probe.kicad_sch")
 		(attr through_hole)
 		(fp_rect
@@
 			(layers "*.Cu" "*.Mask")
 			(remove_unused_layers no)
-			(net 9 "/HV_{L}")
+			(net 9 "/HV_{LIN}")
 			(pintype "passive")
 		)
@@
 			(layers "*.Cu" "*.Mask")
 			(remove_unused_layers no)
-			(net 9 "/HV_{L}")
+			(net 9 "/HV_{LIN}")
 			(pintype "passive")
 		)
@@
 			(layers "F.Cu" "F.Paste" "F.Mask")
 			(roundrect_rratio 0.192308)
-			(net 12 "Net-(J4-Pin_1)")
+			(net 12 "/OUT_{H}")
 			(pintype "passive")
 		)
@@
 			)
 		)
+		(sheetname "Root")
+		(sheetfile "lineScope-05A-probe.kicad_sch")
 		(attr through_hole)
 		(fp_rect
@@
 			(layers "*.Cu" "*.Mask")
 			(remove_unused_layers no)
-			(net 9 "/HV_{L}")
+			(net 9 "/HV_{LIN}")
 			(pintype "passive")
 		)
@@
 			)
 		)
+		(sheetname "Root")
+		(sheetfile "lineScope-05A-probe.kicad_sch")
 		(attr through_hole)
 		(fp_rect
@@
 			(layers "*.Cu" "*.Mask")
 			(remove_unused_layers no)
-			(net 9 "/HV_{L}")
+			(net 9 "/HV_{LIN}")
 			(pintype "passive")
 		)
@@
 			(layers "*.Cu" "*.Mask")
 			(remove_unused_layers no)
-			(net 9 "/HV_{L}")
+			(net 9 "/HV_{LIN}")
 			(pintype "passive")
 		)
@@
 			(layers "*.Cu" "*.Mask")
 			(remove_unused_layers no)
-			(net 12 "Net-(J4-Pin_1)")
+			(net 12 "/OUT_{H}")
 			(pinfunction "Pin_1")
 			(pintype "passive")
@@
 			(layers "*.Cu" "*.Mask")
 			(remove_unused_layers no)
-			(net 11 "Net-(J4-Pin_3)")
+			(net 11 "/OUT_{L}")
 			(pinfunction "Pin_3")
 			(pintype "passive")

Commit message: Fix after bringup 1.0.0
Parts:
- R1: value 300R -> 100R
Other:
- board text added: "Rev 1.1.0 03/2024"
- board text removed: "Rev 1.0.0 03/2024"
Changed lines of the file:
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@@
 	(title_block
 		(title "lineScope 0.5A Probe")
-		(date "2024-03-21")
-		(rev "1.0.0")
+		(date "2024-05-26")
+		(rev "1.1.0")
 		(company "Koszalix")
 	)
@@
 			)
 		)
-		(property "Value" "300R"
+		(property "Value" "100R"
 			(at 0 1.43 90)
 			(layer "F.Fab")
@@
 			)
 		)
-		(property "MPN" "RC0603FR-07300R"
+		(property "MPN" "RC0603FR-07100R"
 			(at 0 0 -90)
 			(unlocked yes)
@@
 		)
 	)
-	(gr_text "Rev 1.0.0 03/2024"
+	(gr_text "Rev 1.1.0 03/2024"
 		(at 103.3 83.3 0)
 		(layer "F.SilkS")
